File: Moving_V4_ESP.kicad_sch (KiCad schematic)
At the start: 46 parts, among them J1 Vin_1, J2 Vin_2, J3 Power_SW, J4 USB_B_Micro, J5 MOTOR_R, J6 Motor_L, SW1 SW_Reset, U1 CH340X, U2 UZ1085L-33-TN3-R, U3 ESP32-WROOM-32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

Commit message: 版を追加
Other:
- title: (none) -> ESP Mini PF base circuit
Changed lines of the file:
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@@
 (kicad_sch (version 20230121) (generator eeschema)
   (paper "A4")
+  (title_block
+    (title "ESP Mini PF base circuit")
+    (date "2025-04-27")
+    (rev "0.1")
+  )
   (junction (at 29.21 50.8) (diameter 0) (color 0 0 0 0)
   )
